File: mounting_holes.kicad_sch (KiCad schematic)
At the start: 4 parts

Commit message: printed pdf from schematics
Signed-off-by: Mika Laitio <lamikr@gmail.com>
Other:
- company: (none) -> Mika Laitio
- title: (none) -> I2S Audio to AES/EBU Optical Toslink
Changed lines of the file:
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@@
   (paper "A4")
   (title_block
+    (title "I2S Audio to AES/EBU Optical Toslink")
     (date "2023-12-26")
     (rev "v0.1")
+    (company "Mika Laitio")
   )
   (text_box "Mounting Holes for PCB"
